File: Eagle/AKS.sch (EAGLE design)
At the start: 13 parts, among them IC1 2982-DRV8825, IC2 2982-DRV8825

Commit message: Eagle
Parts:
- removed C2: 100uF, rcl:CPOL-EUE5-10.5
- removed UV: (no value), HTL22_kontakte:PINHD-1X2
- added X1: (no value), con-ptr500:AK500/2
- C1: value 100uF -> (none); device rcl:CPOL-EUE5-10.5 -> rcl:CPOL-EUE2,5-6E
- IC1, IC2: value 2982-DRV8825 -> 2133-DRV8825; device pololu-stepper-driver:2982-DRV8825 -> pololu-stepper-driver:2133-DRV8825
- renumbered U$3 to U$1
Connections:
- net +40V: now also X1-2.KL; no longer C2.+, UV.1
- net DIR: now also IC2.DIR; no longer IC1.DIR
- net DIR_2: now also IC1.DIR; no longer IC2.DIR
- net ENABLE: now also IC2.!EN; no longer IC1.!EN
- net ENABLE_2: now also IC1.!EN; no longer IC2.!EN
- net GND: no longer U$1.GND@2, U$1.GND@3
- net GND2: now also X1-1.KL; no longer C2.-, UV.2
- net M0: now also IC2.M0; no longer IC1.M0
- net M0_2: now also IC1.M0; no longer IC2.M0
- net M1: now also IC2.M1; no longer IC1.M1
- net M1_2: now also IC1.M1; no longer IC2.M1
- net M2: now also IC2.M2; no longer IC1.M2
- net M2_2: now also IC1.M2; no longer IC2.M2
- net N$1: now also IC2.B2; no longer IC1.B2
- net N$10: now also IC2.A2; no longer IC1.A2
- net N$15: now also SCANNER.1; no longer SCANNER.2
- net N$16: now also SCANNER.2; no longer SCANNER.3
- net N$2: now also IC2.B1; no longer IC1.B1
- net N$3: now also IC2.A1; no longer IC1.A1
- net N$4: now also IC1.B2; no longer IC2.B2
- net N$5: now also IC1.B1; no longer IC2.B1
- net N$6: now also IC1.A1; no longer IC2.A1
- net N$7: now also IC1.A2; no longer IC2.A2
- net N$8: now also U$1.A11
- net N$9: now also U$1.A12
- net STEP: now also IC2.STEP; no longer IC1.STEP
- net STEP_2: now also IC1.STEP; no longer IC2.STEP
- net VCC: now also SCANNER.3; no longer SCANNER.1
Other:
- moved on the sheet: C1, ENDSCHALTER, IC1, IC2, R1, R2, SCANNER
