File: Eagle/AKS.sch (EAGLE design)
At the start: 7 parts, among them IC1 2982-DRV8825

Commit message: nichtsloeschenbitte
Parts:
- removed ARDUINO_NANO1: (no value), ArduinoNanoV30:ARDUINO_NANO
- removed U$1: KY-040, KY-040:KY-040
- removed U$2: 13"OLED13"OLED, 13oled:13"OLED13"OLED
- added C2: 100uF, rcl:CPOL-EUE5-10.5
- added IC2: 2982-DRV8825, pololu-stepper-driver:2982-DRV8825
- added NEMA17_PINS_2: (no value), con-lstb:MA04-1
- added U$3: MEGA_DEVICE, ArduinoMegaOutline:MEGA_DEVICE
- added X2: (no value), con-ptr500:AK500/2-H
Connections:
- removed net CLK: ARDUINO_NANO1.D10, U$1.CLK
- removed net DT: ARDUINO_NANO1.D11, U$1.DT
- removed net SCL: ARDUINO_NANO1.A5, U$2.SCL
- removed net SDA: ARDUINO_NANO1.A4, U$2.SDA
- removed net SW: ARDUINO_NANO1.D12, U$1.SW
- new net DIR_2: IC2.DIR, U$3.27
- new net ENABLE_2: IC2.!EN, U$3.24
- new net M0_2: IC2.M0, U$3.22
- new net M1_2: IC2.M1, U$3.23
- new net M2_2: IC2.M2, U$3.25
- new net N$12: U$3.GND@1
- new net N$4: IC2.B2, NEMA17_PINS_2.1
- new net N$5: IC2.B1, NEMA17_PINS_2.2
- new net N$6: IC2.A1, NEMA17_PINS_2.3
- new net N$7: IC2.A2, NEMA17_PINS_2.4
- new net N$8: U$3.20, X2-2.KL
- new net N$9: U$3.21, X2-1.KL
- new net STEP_2: IC2.STEP, U$3.29
- net +40V: now also C2.+, IC2.VMOT
- net DIR: now also U$3.0; no longer ARDUINO_NANO1.D2
- net ENABLE: now also U$3.5; no longer ARDUINO_NANO1.D4
- net GND: now also IC2.GND1, U$3.GND@2, U$3.GND@3; no longer ARDUINO_NANO1.GND@1, ARDUINO_NANO1.GND@2, U$1.GND, U$2.GND
- net GND2: now also C2.-, IC2.GND2
- net M0: now also U$3.4; no longer ARDUINO_NANO1.D5
- net M1: now also U$3.3; no longer ARDUINO_NANO1.D6
- net M2: now also U$3.2; no longer ARDUINO_NANO1.D7
- net STEP: now also U$3.1; no longer ARDUINO_NANO1.D3
- net VCC: now also IC2.!RST, IC2.!SLP, U$3.5V; no longer ARDUINO_NANO1.5V, U$1.VCC, U$2.VCC
Other:
- moved on the sheet: C1, IC1, NEMA17_PINS, X1-1, X1-2

Commit message: schematic_update
Parts:
- removed X1: (no value), con-ptr500:AK500/2-H
- added R1, R2: 10k, rcl:R-EU_R1206
- added X4: (no value), HTL22_kontakte:PINHD-1X4
- X2: device con-ptr500:AK500/2-H -> HTL22_kontakte:PINHD-1X2
Connections:
- removed net N$11: IC1.A2, NEMA17_PINS.4
- removed net N$12: U$3.GND@1
- new net N$10: IC1.A2, NEMA17_PINS.2
- net +40V: no longer X1-2.KL
- net DIR: no longer U$3.0
- net DIR_2: no longer U$3.27
- net ENABLE: no longer U$3.5
- net ENABLE_2: now also U$3.0; no longer U$3.24
- net GND: now also R1.1, R2.1
- net GND2: no longer X1-1.KL
- net M0: no longer U$3.4
- net M0_2: no longer U$3.22
- net M1: no longer U$3.3
- net M1_2: now also U$3.2; no longer U$3.23
- net M2: no longer U$3.2
- net M2_2: now also U$3.3; no longer U$3.25
- net N$2: now also NEMA17_PINS.3; no longer NEMA17_PINS.2
- net N$3: now also NEMA17_PINS.4; no longer NEMA17_PINS.3
- net N$5: now also NEMA17_PINS_2.3; no longer NEMA17_PINS_2.2
- net N$6: now also NEMA17_PINS_2.4; no longer NEMA17_PINS_2.3
- net N$7: now also NEMA17_PINS_2.2; no longer NEMA17_PINS_2.4
- net N$8: now also R2.2, X4.1; no longer U$3.20, X2-2.KL
- net N$9: now also R1.2, X4.2; no longer U$3.21, X2-1.KL
- net STEP: no longer U$3.1
- net STEP_2: no longer U$3.29
- net VCC: now also X4.3, X4.4

Commit message: update_w_display
Parts:
- added X1: (no value), HTL22_kontakte:PINHD-1X4
Connections:
- new net N$13: U$3.21, X1.1
- new net N$14: U$3.20, X1.2
- net GND: now also X1.4
- net VCC: now also X1.3
Changed lines of the file:
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@@
 <part name="X4" library="HTL22_kontakte" deviceset="PINHD-1X4" device=""/>
 <part name="X2" library="HTL22_kontakte" deviceset="PINHD-1X2" device=""/>
+<part name="X1" library="HTL22_kontakte" deviceset="PINHD-1X4" device=""/>
 </parts>
 <sheets>
@@
 <instance part="X4" gate="A" x="144.78" y="148.59"/>
 <instance part="X2" gate="G$1" x="257.81" y="144.78"/>
+<instance part="X1" gate="A" x="144.78" y="130.81"/>
 </instances>
 <busses>
@@
 <wire x1="135.89" y1="146.05" x2="129.54" y2="146.05" width="0.1524" layer="91"/>
 <label x="129.54" y="146.05" size="1.016" layer="95" rot="R180" xref="yes"/>
+</segment>
+<segment>
+<pinref part="X1" gate="A" pin="3"/>
+<wire x1="142.24" y1="130.81" x2="135.89" y2="130.81" width="0.1524" layer="91"/>
+<label x="135.89" y="130.81" size="1.016" layer="95" rot="R180" xref="yes"/>
 </segment>
 </net>
@@
 <pinref part="R2" gate="G$1" pin="1"/>
 <wire x1="115.57" y1="139.7" x2="115.57" y2="140.97" width="0.1524" layer="91"/>
+</segment>
+<segment>
+<pinref part="X1" gate="A" pin="4"/>
+<wire x1="142.24" y1="128.27" x2="135.89" y2="128.27" width="0.1524" layer="91"/>
+<label x="135.89" y="128.27" size="1.016" layer="95" rot="R180" xref="yes"/>
 </segment>
 </net>
@@
 </segment>
 </net>
+<net name="N$13" class="0">
+<segment>
+<pinref part="X1" gate="A" pin="1"/>
+<wire x1="142.24" y1="135.89" x2="111.76" y2="135.89" width="0.1524" layer="91"/>
+<pinref part="U$3" gate="G$1" pin="21"/>
+<wire x1="111.76" y1="135.89" x2="111.76" y2="125.73" width="0.1524" layer="91"/>
+</segment>
+</net>
+<net name="N$14" class="0">
+<segment>
+<pinref part="X1" gate="A" pin="2"/>
+<wire x1="142.24" y1="133.35" x2="109.22" y2="133.35" width="0.1524" layer="91"/>
+<pinref part="U$3" gate="G$1" pin="20"/>
+<wire x1="109.22" y1="133.35" x2="109.22" y2="125.73" width="0.1524" layer="91"/>
+</segment>
+</net>

Commit message: updated_schematic
Parts:
- added SCANNER: (no value), HTL22_kontakte:PINHD-1X4
- renumbered X1 to DISPLAY, X2 to UV, X4 to ENDSCHALTER
Connections:
- new net N$11: U$3.6
- new net N$12: U$3.7
- new net N$15: SCANNER.2, U$3.19
- new net N$16: SCANNER.3, U$3.18
- net +40V: now also UV.1
- net DIR: now also U$3.13
- net DIR_2: now also U$3.5
- net ENABLE: now also U$3.8
- net GND: now also SCANNER.4
- net GND2: now also UV.2
- net M0: now also U$3.9
- net M0_2: now also U$3.1
- net M1: now also U$3.10
- net M2: now also U$3.11
- net N$13: now also U$3.20; no longer U$3.21
- net N$14: now also U$3.21; no longer U$3.20
- net STEP: now also U$3.12
- net STEP_2: now also U$3.4
- net VCC: now also SCANNER.1
Changed lines of the file:
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@@
 <part name="R2" library="rcl" deviceset="R-EU_" device="R1206" value="10k"/>
 <part name="GND4" library="supply1" deviceset="GND" device=""/>
-<part name="X4" library="HTL22_kontakte" deviceset="PINHD-1X4" device=""/>
-<part name="X2" library="HTL22_kontakte" deviceset="PINHD-1X2" device=""/>
-<part name="X1" library="HTL22_kontakte" deviceset="PINHD-1X4" device=""/>
+<part name="ENDSCHALTER" library="HTL22_kontakte" deviceset="PINHD-1X4" device=""/>
+<part name="UV" library="HTL22_kontakte" deviceset="PINHD-1X2" device=""/>
+<part name="DISPLAY" library="HTL22_kontakte" deviceset="PINHD-1X4" device=""/>
+<part name="SCANNER" library="HTL22_kontakte" deviceset="PINHD-1X4" device=""/>
 </parts>
 <sheets>
@@
 <attribute name="VALUE" x="113.03" y="134.62" size="1.778" layer="96"/>
 </instance>
-<instance part="X4" gate="A" x="144.78" y="148.59"/>
-<instance part="X2" gate="G$1" x="257.81" y="144.78"/>
-<instance part="X1" gate="A" x="144.78" y="130.81"/>
+<instance part="ENDSCHALTER" gate="A" x="144.78" y="148.59"/>
+<instance part="UV" gate="G$1" x="257.81" y="144.78"/>
+<instance part="DISPLAY" gate="A" x="144.78" y="130.81"/>
+<instance part="SCANNER" gate="A" x="144.78" y="114.3"/>
 </instances>
 <busses>
@@
 </segment>
 <segment>
-<pinref part="X4" gate="A" pin="3"/>
+<pinref part="ENDSCHALTER" gate="A" pin="3"/>
 <wire x1="142.24" y1="148.59" x2="135.89" y2="148.59" width="0.1524" layer="91"/>
-<pinref part="X4" gate="A" pin="4"/>
+<pinref part="ENDSCHALTER" gate="A" pin="4"/>
 <wire x1="135.89" y1="148.59" x2="135.89" y2="146.05" width="0.1524" layer="91"/>
 <wire x1="135.89" y1="146.05" x2="142.24" y2="146.05" width="0.1524" layer="91"/>
@@
 </segment>
 <segment>
-<pinref part="X1" gate="A" pin="3"/>
+<pinref part="DISPLAY" gate="A" pin="3"/>
 <wire x1="142.24" y1="130.81" x2="135.89" y2="130.81" width="0.1524" layer="91"/>
 <label x="135.89" y="130.81" size="1.016" layer="95" rot="R180" xref="yes"/>
+</segment>
+<segment>
+<pinref part="SCANNER" gate="A" pin="1"/>
+<wire x1="142.24" y1="119.38" x2="135.89" y2="119.38" width="0.1524" layer="91"/>
+<label x="135.89" y="119.38" size="1.016" layer="95" rot="R180" xref="yes"/>
 </segment>
 </net>
@@
 </segment>
 <segment>
-<wire x1="67.31" y1="130.81" x2="67.31" y2="134.62" width="0.1524" layer="91"/>
 <label x="67.31" y="134.62" size="1.016" layer="95" rot="R90" xref="yes"/>
+<pinref part="U$3" gate="G$1" pin="8"/>
+<wire x1="67.31" y1="134.62" x2="67.31" y2="125.73" width="0.1524" layer="91"/>
 </segment>
 </net>
@@
 <wire x1="243.84" y1="88.9" x2="243.84" y2="144.78" width="0.1524" layer="91"/>
 <junction x="243.84" y="144.78"/>
+<pinref part="UV" gate="G$1" pin="2"/>
 </segment>
 </net>
@@
 </segment>
 <segment>
-<wire x1="54.61" y1="130.81" x2="54.61" y2="134.62" width="0.1524" layer="91"/>
 <label x="54.61" y="134.62" size="1.016" layer="95" rot="R90" xref="yes"/>
+<pinref part="U$3" gate="G$1" pin="13"/>
+<wire x1="54.61" y1="134.62" x2="54.61" y2="125.73" width="0.1524" layer="91"/>
 </segment>
 </net>
@@
 </segment>
 <segment>
-<wire x1="57.15" y1="130.81" x2="57.15" y2="134.62" width="0.1524" layer="91"/>
 <label x="57.15" y="134.62" size="1.016" layer="95" rot="R90" xref="yes"/>
+<pinref part="U$3" gate="G$1" pin="12"/>
+<wire x1="57.15" y1="134.62" x2="57.15" y2="125.73" width="0.1524" layer="91"/>
 </segment>
 </net>
@@
 </segment>
 <segment>
-<wire x1="64.77" y1="130.81" x2="64.77" y2="134.62" width="0.1524" layer="91"/>
 <label x="64.77" y="134.62" size="1.016" layer="95" rot="R90" xref="yes"/>
+<pinref part="U$3" gate="G$1" pin="9"/>
+<wire x1="64.77" y1="134.62" x2="64.77" y2="125.73" width="0.1524" layer="91"/>
 </segment>
 </net>
@@
 </segment>
 <segment>
-<wire x1="62.23" y1="130.81" x2="62.23" y2="134.62" width="0.1524" layer="91"/>
 <label x="62.23" y="134.62" size="1.016" layer="95" rot="R90" xref="yes"/>
+<wire x1="62.23" y1="134.62" x2="62.23" y2="125.73" width="0.1524" layer="91"/>
+<pinref part="U$3" gate="G$1" pin="10"/>
 </segment>
 </net>
@@
 </segment>
 <segment>
-<wire x1="59.69" y1="130.81" x2="59.69" y2="134.62" width="0.1524" layer="91"/>
 <label x="59.69" y="134.62" size="1.016" layer="95" rot="R90" xref="yes"/>
+<pinref part="U$3" gate="G$1" pin="11"/>
+<wire x1="59.69" y1="134.62" x2="59.69" y2="125.73" width="0.1524" layer="91"/>
 </segment>
 </net>
@@
 </segment>
 <segment>
-<pinref part="X1" gate="A" pin="4"/>
+<pinref part="DISPLAY" gate="A" pin="4"/>
 <wire x1="142.24" y1="128.27" x2="135.89" y2="128.27" width="0.1524" layer="91"/>
 <label x="135.89" y="128.27" size="1.016" layer="95" rot="R180" xref="yes"/>
+</segment>
+<segment>
+<pinref part="SCANNER" gate="A" pin="4"/>
+<wire x1="142.24" y1="111.76" x2="135.89" y2="111.76" width="0.1524" layer="91"/>
+<label x="135.89" y="111.76" size="1.016" layer="95" rot="R180" xref="yes"/>
 </segment>
 </net>
@@
 <wire x1="238.76" y1="93.98" x2="215.9" y2="93.98" width="0.1524" layer="91"/>
 <junction x="238.76" y="147.32"/>
+<pinref part="UV" gate="G$1" pin="1"/>
 </segment>
 </net>
@@
 </segment>
 <segment>
-<wire x1="86.36" y1="130.81" x2="86.36" y2="134.62" width="0.1524" layer="91"/>
 <label x="86.36" y="134.62" size="1.016" layer="95" rot="R90" xref="yes"/>
+<pinref part="U$3" gate="G$1" pin="1"/>
+<wire x1="86.36" y1="134.62" x2="86.36" y2="125.73" width="0.1524" layer="91"/>
 </segment>
 </net>
@@
 </segment>
 <segment>
-<wire x1="78.74" y1="130.81" x2="78.74" y2="134.62" width="0.1524" layer="91"/>
 <label x="78.74" y="134.62" size="1.016" layer="95" rot="R90" xref="yes"/>
+<pinref part="U$3" gate="G$1" pin="4"/>
+<wire x1="78.74" y1="134.62" x2="78.74" y2="125.73" width="0.1524" layer="91"/>
 </segment>
 </net>
@@
 </segment>
 <segment>
-<wire x1="76.2" y1="130.81" x2="76.2" y2="134.62" width="0.1524" layer="91"/>
 <label x="76.2" y="134.62" size="1.016" layer="95" rot="R90" xref="yes"/>
+<pinref part="U$3" gate="G$1" pin="5"/>
+<wire x1="76.2" y1="134.62" x2="76.2" y2="125.73" width="0.1524" layer="91"/>
 </segment>
 </net>
@@
 <wire x1="115.57" y1="151.13" x2="115.57" y2="153.67" width="0.1524" layer="91"/>
 <junction x="115.57" y="153.67"/>
-<pinref part="X4" gate="A" pin="1"/>
+<pinref part="ENDSCHALTER" gate="A" pin="1"/>
 <wire x1="115.57" y1="153.67" x2="142.24" y2="153.67" width="0.1524" layer="91"/>
 </segment>
@@
 <pinref part="R1" gate="G$1" pin="2"/>
 <junction x="101.6" y="148.59"/>
-<pinref part="X4" gate="A" pin="2"/>
+<pinref part="ENDSCHALTER" gate="A" pin="2"/>
 <wire x1="142.24" y1="151.13" x2="101.6" y2="151.13" width="0.1524" layer="91"/>
 <wire x1="101.6" y1="151.13" x2="101.6" y2="148.59" width="0.1524" layer="91"/>
@@
 <net name="N$11" class="0">
 <segment>
-<wire x1="73.66" y1="130.81" x2="73.66" y2="134.62" width="0.1524" layer="91"/>
+<pinref part="U$3" gate="G$1" pin="6"/>
+<wire x1="73.66" y1="134.62" x2="73.66" y2="125.73" width="0.1524" layer="91"/>
 </segment>
 </net>
 <net name="N$12" class="0">
 <segment>
-<wire x1="71.12" y1="130.81" x2="71.12" y2="134.62" width="0.1524" layer="91"/>
+<pinref part="U$3" gate="G$1" pin="7"/>
+<wire x1="71.12" y1="134.62" x2="71.12" y2="125.73" width="0.1524" layer="91"/>
 </segment>
 </net>
 <net name="N$13" class="0">
 <segment>
-<pinref part="X1" gate="A" pin="1"/>
-<wire x1="142.24" y1="135.89" x2="111.76" y2="135.89" width="0.1524" layer="91"/>
+<pinref part="DISPLAY" gate="A" pin="1"/>
+<wire x1="142.24" y1="135.89" x2="109.22" y2="135.89" width="0.1524" layer="91"/>
+<pinref part="U$3" gate="G$1" pin="20"/>
+<wire x1="109.22" y1="135.89" x2="109.22" y2="125.73" width="0.1524" layer="91"/>
+</segment>
+</net>
+<net name="N$14" class="0">
+<segment>
 <pinref part="U$3" gate="G$1" pin="21"/>
-<wire x1="111.76" y1="135.89" x2="111.76" y2="125.73" width="0.1524" layer="91"/>
-</segment>
-</net>
-<net name="N$14" class="0">
-<segment>
-<pinref part="X1" gate="A" pin="2"/>
-<wire x1="142.24" y1="133.35" x2="109.22" y2="133.35" width="0.1524" layer="91"/>
-<pinref part="U$3" gate="G$1" pin="20"/>
-<wire x1="109.22" y1="133.35" x2="109.22" y2="125.73" width="0.1524" layer="91"/>
-</segment>
-</net>
+<pinref part="DISPLAY" gate="A" pin="2"/>
+<wire x1="111.76" y1="125.73" x2="111.76" y2="133.35" width="0.1524" layer="91"/>
+<wire x1="111.76" y1="133.35" x2="142.24" y2="133.35" width="0.1524" layer="91"/>
+</segment>
+</net>
+<net name="N$15" class="0">
+<segment>
+<pinref part="SCANNER" gate="A" pin="2"/>
+<wire x1="142.24" y1="116.84" x2="106.68" y2="116.84" width="0.1524" layer="91"/>
+<pinref part="U$3" gate="G$1" pin="19"/>
+<wire x1="106.68" y1="116.84" x2="106.68" y2="125.73" width="0.1524" layer="91"/>
+</segment>
+</net>
+<net name="N$16" class="0">
+<segment>
+<pinref part="SCANNER" gate="A" pin="3"/>
+<wire x1="142.24" y1="114.3" x2="104.14" y2="114.3" width="0.1524" layer="91"/>
+<pinref part="U$3" gate="G$1" pin="18"/>
+<wire x1="104.14" y1="114.3" x2="104.14" y2="125.73" width="0.1524" layer="91"/>
+</segment>
+</net>

Commit message: hmmmm
Parts:
- removed C2: 100uF, rcl:CPOL-EUE5-10.5
- removed UV: (no value), HTL22_kontakte:PINHD-1X2
- added X1: (no value), con-ptr500:AK500/2
- C1: value 100uF -> (none); device rcl:CPOL-EUE5-10.5 -> rcl:CPOL-EUE2,5-6E
Connections:
- removed net +40V: C1.+, C2.+, IC1.VMOT, IC2.VMOT, UV.1
- removed net N$9: ENDSCHALTER.2, R1.2
- new net +25V: C1.+, IC1.VMOT, IC2.VMOT, X1-2.KL
- new net N$17: ENDSCHALTER.4, R1.2, U$3.A15
- net GND: now also U$3.GND@1
- net GND2: now also X1-1.KL; no longer C2.-, UV.2
- net N$15: now also SCANNER.1; no longer SCANNER.2
- net N$16: now also SCANNER.2; no longer SCANNER.3
- net N$8: now also ENDSCHALTER.2, U$3.A14; no longer ENDSCHALTER.1
- net VCC: now also ENDSCHALTER.1, SCANNER.3; no longer ENDSCHALTER.4, SCANNER.1
Other:
- moved on the sheet: C1, ENDSCHALTER, R1, R2, SCANNER
