File: Eagle/AKS.brd (EAGLE design)
At the start: 110 x 80 mm, 9 parts, among them IC1 2982-DRV8825, IC2 2982-DRV8825

Commit message: schematic_update
Parts:
- removed X1: (no value), con-ptr500:AK500/2-H
- added R1, R2: 10k, rcl:R1206
- added X4: (no value), HTL22_kontakte:1X04
- X2: device con-ptr500:AK500/2-H -> HTL22_kontakte:1X02
- moved X2 125.7 mm to (5.08, -64.1), turned to 0 degrees
Connections:
- removed net N$11: IC1.11, NEMA17_PINS.4
- removed net N$12: U$3.GND@1
- new net N$10: IC1.11, NEMA17_PINS.2
- net +40V: no longer X1.2
- net DIR: no longer U$3.0
- net DIR_2: no longer U$3.27
- net ENABLE: no longer U$3.5
- net ENABLE_2: now also U$3.0; no longer U$3.24
- net GND: now also R1.1, R2.1
- net GND2: no longer X1.1
- net M0: no longer U$3.4
- net M0_2: no longer U$3.22
- net M1: no longer U$3.3
- net M1_2: now also U$3.2; no longer U$3.23
- net M2: no longer U$3.2
- net M2_2: now also U$3.3; no longer U$3.25
- net N$2: now also NEMA17_PINS.3; no longer NEMA17_PINS.2
- net N$3: now also NEMA17_PINS.4; no longer NEMA17_PINS.3
- net N$5: now also NEMA17_PINS_2.3; no longer NEMA17_PINS_2.2
- net N$6: now also NEMA17_PINS_2.4; no longer NEMA17_PINS_2.3
- net N$7: now also NEMA17_PINS_2.2; no longer NEMA17_PINS_2.4
- net N$8: now also R2.2, X4.1; no longer U$3.20, X2.2
- net N$9: now also R1.2, X4.2; no longer U$3.21, X2.1
- net STEP: no longer U$3.1
- net STEP_2: no longer U$3.29
- net VCC: now also X4.3, X4.4
Routing:
- net N$9: track 99.0 -> 0.00 mm
- net N$8: track 96.4 -> 0.00 mm
- net GND2: track 131.8 -> 105.8 mm
- net STEP_2: track 39.7 -> 30.8 mm
- net STEP: track 7.62 -> 0.00 mm
- net DIR: track 7.62 -> 0.00 mm
- net DIR_2: track 26.5 -> 19.5 mm
- net M2: track 12.0 -> 6.88 mm
- net N$7: track 4.44 -> 0.00 mm
- net N$6: track 4.44 -> 0.00 mm
- net N$5: track 4.44 -> 0.00 mm
- net N$3: track 4.44 -> 0.00 mm
- net N$2: track 4.44 -> 0.00 mm
- net N$11: track 4.44 -> 0.00 mm
- net N$1: track 4.44 -> 0.00 mm
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
Commit message: update_w_display
Parts:
- added X1: (no value), HTL22_kontakte:1X04
Connections:
- new net N$13: U$3.21, X1.1
- new net N$14: U$3.20, X1.2
- net GND: now also X1.4
- net VCC: now also X1.3
Changed lines of the file:
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@@
 <element name="X4" library="HTL22_kontakte" package="1X04" value="" x="7.62" y="-48.895"/>
 <element name="X2" library="HTL22_kontakte" package="1X02" value="" x="5.08" y="-64.135"/>
+<element name="X1" library="HTL22_kontakte" package="1X04" value="" x="7.62" y="-79.375"/>
 </elements>
 <signals>
@@
 <contactref element="X4" pad="3"/>
 <contactref element="X4" pad="4"/>
+<contactref element="X1" pad="3"/>
 <wire x1="39.37" y1="3.81" x2="57.15" y2="59.69" width="0" layer="19" extent="1-1"/>
 <wire x1="11.43" y1="-48.895" x2="39.37" y2="3.81" width="0" layer="19" extent="1-1"/>
 <wire x1="8.89" y1="-48.895" x2="11.43" y2="-48.895" width="0" layer="19" extent="1-1"/>
+<wire x1="8.89" y1="-79.375" x2="8.89" y2="-48.895" width="0" layer="19" extent="1-1"/>
 </signal>
 <signal name="ENABLE">
@@
 <contactref element="R1" pad="1"/>
 <contactref element="R2" pad="1"/>
+<contactref element="X1" pad="4"/>
 <wire x1="64.77" y1="72.39" x2="101.6" y2="72.39" width="0" layer="19" extent="1-1"/>
 <wire x1="44.45" y1="3.81" x2="64.77" y2="72.39" width="0" layer="19" extent="1-1"/>
@@
 <wire x1="-2.692" y1="-11.43" x2="41.91" y2="3.81" width="0" layer="19" extent="1-1"/>
 <wire x1="-2.692" y1="-17.78" x2="-2.692" y2="-11.43" width="0" layer="19" extent="1-1"/>
+<wire x1="11.43" y1="-79.375" x2="-2.692" y2="-17.78" width="0" layer="19" extent="1-1"/>
 </signal>
 <signal name="+40V">
@@
 <wire x1="0.152" y1="-11.43" x2="6.35" y2="-48.895" width="0" layer="19" extent="1-1"/>
 </signal>
+<signal name="N$13">
+<contactref element="X1" pad="1"/>
+<contactref element="U$3" pad="21"/>
+<wire x1="3.81" y1="-79.375" x2="87.63" y2="52.07" width="0" layer="19" extent="1-1"/>
+</signal>
+<signal name="N$14">
+<contactref element="X1" pad="2"/>
+<contactref element="U$3" pad="20"/>
+<wire x1="6.35" y1="-79.375" x2="85.09" y2="52.07" width="0" layer="19" extent="1-1"/>
+</signal>
 </signals>

Commit message: updated_schematic
Parts:
- removed X1, X4: (no value), HTL22_kontakte:1X04
- removed X2: (no value), HTL22_kontakte:1X02
- added DISPLAY, ENDSCHALTER, SCANNER: (no value), HTL22_kontakte:1X04
- added UV: (no value), HTL22_kontakte:1X02
- moved NEMA17_PINS_2 107.2 mm to (6.35, 13.3), turned to 90 degrees
- moved NEMA17_PINS 70.9 mm to (6.35, 26.0), turned to 90 degrees
- moved R2 58.1 mm to (12.1, 38.7), turned to 180 degrees
- moved R1 54.4 mm to (12.1, 41.3), turned to 180 degrees
- moved C2 53.9 mm to (39.4, 26.0), turned to 180 degrees
- moved C1 49.2 mm to (66.0, 26.0), turned to 180 degrees
- moved IC2 43.1 mm to (58.4, 40.0), turned to 270 degrees
- moved IC1 35.5 mm to (31.8, 40.0), turned to 270 degrees
- moved U$3 2.84 mm to (49.5, 26.7)
Connections:
- new net N$11: U$3.6
- new net N$12: U$3.7
- new net N$15: SCANNER.2, U$3.19
- new net N$16: SCANNER.3, U$3.18
- net +40V: now also UV.1
- net DIR: now also U$3.13
- net DIR_2: now also U$3.5
- net ENABLE: now also U$3.8
- net GND: now also DISPLAY.4, SCANNER.4; no longer X1.4
- net GND2: now also UV.2
- net M0: now also U$3.9
- net M0_2: now also U$3.1
- net M1: now also U$3.10
- net M2: now also U$3.11
- net N$13: now also DISPLAY.1, U$3.20; no longer U$3.21, X1.1
- net N$14: now also DISPLAY.2, U$3.21; no longer U$3.20, X1.2
- net N$8: now also ENDSCHALTER.1; no longer X4.1
- net N$9: now also ENDSCHALTER.2; no longer X4.2
- net STEP: now also U$3.12
- net STEP_2: now also U$3.4
- net VCC: now also DISPLAY.3, ENDSCHALTER.3, ENDSCHALTER.4, SCANNER.1; no longer X1.3, X4.3, X4.4
Routing:
- net GND: track 0.00 -> 178.1 mm, vias 0 -> 6
- net VCC: track 43.5 -> 176.8 mm
- net N$4: track 4.44 -> 80.3 mm
- net N$7: track 0.00 -> 74.0 mm
- net N$5: track 0.00 -> 72.2 mm
- net N$6: track 0.00 -> 66.6 mm
- net N$1: track 0.00 -> 38.4 mm
- net N$10: track 0.00 -> 36.6 mm
- net N$2: track 0.00 -> 31.2 mm
- net N$14: track 0.00 -> 29.7 mm
- net N$3: track 0.00 -> 27.2 mm
- net STEP_2: track 30.8 -> 4.45 mm
- net N$13: track 0.00 -> 24.7 mm
- net GND2: track 105.8 -> 87.3 mm
- net M2_2: track 24.2 -> 6.92 mm
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Other:
- board size 110 x 80 mm -> 100 x 54 mm

Commit message: hmmmm
Parts:
- removed C2: 100uF, rcl:E5-10,5
- removed UV: (no value), HTL22_kontakte:1X02
- added X1: (no value), con-ptr500:AK500/2
- C1: value 100uF -> (none); device rcl:E5-10,5 -> rcl:E2,5-6E
- moved ENDSCHALTER 84.7 mm to (83.8, 8.26), turned to 0 degrees
- moved R1 80.3 mm to (87.6, 14.0), turned to 270 degrees
- moved R2 74.7 mm to (82.5, 14.0), turned to 270 degrees
- moved NEMA17_PINS_2 54.6 mm to (61.0, 11.4), turned to 180 degrees
- moved NEMA17_PINS 43.2 mm to (47.0, 11.4), turned to 180 degrees
- moved C1 25.5 mm to (45.1, 40.6), turned to 270 degrees
- moved DISPLAY 9.44 mm to (85.7, 31.8)
- moved SCANNER 6.38 mm to (76.2, 40.6)
Connections:
- removed net +40V: C1.+, C2.+, IC1.16, IC2.16, UV.1
- removed net N$9: ENDSCHALTER.2, R1.2
- new net +25V: C1.+, IC1.16, IC2.16, X1.2
- new net N$17: ENDSCHALTER.4, R1.2, U$3.A15
- net GND: now also U$3.GND@1
- net GND2: now also X1.1; no longer C2.-, UV.2
- net N$15: now also SCANNER.1; no longer SCANNER.2
- net N$16: now also SCANNER.2; no longer SCANNER.3
- net N$8: now also ENDSCHALTER.2, U$3.A14; no longer ENDSCHALTER.1
- net VCC: now also ENDSCHALTER.1, SCANNER.3; no longer ENDSCHALTER.4, SCANNER.1
Routing:
- net GND: track 178.1 -> 2.54 mm, vias 6 -> 0
- net +40V: track 81.8 -> 0.00 mm
- net +25V: track 0.00 -> 72.5 mm
- net N$4: track 80.3 -> 23.3 mm
- net N$5: track 72.2 -> 22.2 mm
- net N$6: track 66.6 -> 22.2 mm
- net N$7: track 74.0 -> 35.5 mm
- net GND2: track 87.3 -> 72.1 mm, vias 2 -> 0
- net N$17: track 0.00 -> 11.8 mm
- net VCC: track 176.8 -> 165.2 mm
- net N$8: track 4.29 -> 14.3 mm
- net N$10: track 36.6 -> 44.6 mm
- net N$13: track 24.7 -> 17.3 mm
- net N$14: track 29.7 -> 22.4 mm
- net N$3: track 27.2 -> 32.7 mm
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- added copper zone on layer 1, net GND
Other:
- board size 100 x 54 mm -> 101 x 53.3 mm
